File: ThermoBuzzer_pcb/ThermoBuzzer_pcb.kicad_sch (KiCad schematic)
At the start: 6 parts, among them SW1 SW_Push

Commit message: Further work on Schematics + parts
Parts:
- removed C1: C, symbol Device:C
- added R2: 100k, symbol Device:R
- R1: value R -> 100
Connections:
- net at BZ1.1 (+): now also A1.8 (D5)
- net at BZ1.2 (-): now also A1.4 (GND), R1.1
- net at A1.19 (A0): now also TH1.2, R2.1
- net at A1.2 (D0/RX): now also R1.2, SW1.2
- net at A1.27 (+5V): now also SW1.1, TH1.1
- net at A1.29 (GND): now also R2.2
Other:
- title: (none) -> Thermobuzzer
- moved on the sheet: BZ1, R1, SW1, TH1

Commit message: Finalize arduino + temperature
Parts:
- added A2: Arduino_Nano_v2.x, Module:Arduino_Nano, symbol MCU_Module:Arduino_Nano_v2.x
- added BZ2: Buzzer, symbol Device:Buzzer
- added R3: 100, symbol Device:R
- added SW2: SW_Push, symbol Switch:SW_Push
- added U1: ~, symbol thermosensor:BME280_new
Connections:
- new net: A2.4 (GND), BZ2.2 (-), R3.1
- new net: A2.2 (D0/RX), R3.2, SW2.2
- new net: A2.8 (D5), BZ2.1 (+)
- new net: A2.17 (3V3), U1.1 (VIN)
- new net: A2.29 (GND), U1.2 (GND)
- new net: A2.24 (A5), U1.3 (SCL)
- new net: A2.23 (A4), U1.4 (SDA)
- new net: A2.27 (+5V), SW2.1
