File: ThermoBuzzer_pcb/ThermoBuzzer_v2_pcb.kicad_sch (KiCad schematic)
At the start: 8 parts, among them SW2 SW_Push

Commit message: april 4 schematic + footprints
Parts:
- removed R4: 100k, Resistor_THT:R_Axial_DIN0207_L6.3mm_D2.5mm_P7.62mm_Horizontal, symbol Device:R
- removed TH2: Thermistor, symbol Device:Thermistor
- added A1: Arduino_Nano_v2.x, Module:Arduino_Nano, symbol MCU_Module:Arduino_Nano_v2.x
- added BZ1: Buzzer, symbol Device:Buzzer
- added R1: 100, symbol Device:R
- added R2: 100k, symbol Device:R
- added SW1: SW_Push, symbol Switch:SW_Push
- added TH1: Thermistor, symbol Device:Thermistor
- BT1: footprint Resistor_THT:R_Axial_DIN0204_L3.6mm_D1.6mm_P1.90mm_Vertical -> (none)
- R3: footprint Resistor_THT:R_Axial_DIN0207_L6.3mm_D2.5mm_P7.62mm_Horizontal -> (none)
Connections:
- net +9V: now also A1.30 (VIN)
- net GND: now also A1.4 (GND), BZ1.2 (-), R1.1
- new net: A1.8 (D5), BZ1.1 (+)
- new net: A1.19 (A0), R2.1, TH1.2
- new net: A1.2 (D0/RX), R1.2, SW1.2
- new net: A1.27 (+5V), SW1.1, TH1.1
- new net: A1.29 (GND), R2.2
Other:
- moved on the sheet: A2, BT1, BZ2, R3, SW2, U1

Commit message: 4.15
Parts:
- added A3: Arduino_Nano_v2.x, Module:Arduino_Nano, symbol MCU_Module:Arduino_Nano_v2.x
- added BT2: Battery_Cell, Resistor_THT:R_Axial_DIN0204_L3.6mm_D1.6mm_P1.90mm_Vertical, symbol Device:Battery_Cell
- added BZ3: Buzzer, symbol Device:Buzzer
- added R4: 100k, Resistor_THT:R_Axial_DIN0207_L6.3mm_D2.5mm_P7.62mm_Horizontal, symbol Device:R
- added R4: 100, Resistor_THT:R_Axial_DIN0207_L6.3mm_D2.5mm_P7.62mm_Horizontal, symbol Device:R
- added SW3: SW_Push, symbol Switch:SW_Push
- added TH2: Thermistor, symbol Device:Thermistor
- added U2: ~, symbol thermosensor:BME280_new
Connections:
- net +9V: now also A3.30 (VIN), BT2.1 (+)
- net GND: now also A3.4 (GND), BT2.2 (-), BZ3.2 (-), R4.1
- new net: A3.17 (3V3), U2.1 (VIN)
- new net: A3.19 (A0), R4.1, TH2.2
- new net: A3.2 (D0/RX), R4.2, SW3.2
- new net: A3.23 (A4), U2.4 (SDA)
- new net: A3.24 (A5), U2.3 (SCL)
- new net: A3.27 (+5V), SW3.1, TH2.1
- new net: A3.29 (GND), R4.2, U2.2 (GND)
- new net: A3.8 (D5), BZ3.1 (+)
Other:
- moved on the sheet: A1, BZ1, R1, R2, SW1, TH1
