File: ThermoBuzzer_pcb/ThermoBuzzer_pcb.kicad_pcb (KiCad board)
At the start: 2 copper layers, 17.8 x 33 mm, 7 parts

Commit message: 4.18
Parts:
- added BME280: ~, custom_footprints:AHT20+BMP280, F.Cu at (112.8, 97.2)
- added BT2: Battery_Cell, Resistor_THT:R_Axial_DIN0204_L3.6mm_D1.6mm_P1.90mm_Vertical, F.Cu at (92.7, 70.1)
- added BZ1: Buzzer, Buzzer_Beeper:Buzzer_12x9.5RM7.6, F.Cu at (61.5, 103.7)
- added R1: 100, Resistor_THT:R_Axial_DIN0207_L6.3mm_D2.5mm_P7.62mm_Horizontal, F.Cu at (64.6, 91.0)
- added R2: 100k, Resistor_THT:R_Axial_DIN0207_L6.3mm_D2.5mm_P7.62mm_Horizontal, F.Cu at (101.4, 109.1)
- added SW1: SW_Push, Button_Switch_THT:SW_PUSH_6mm, F.Cu at (58.7, 78.2)
- added TH1: Thermistor, Resistor_THT:R_Axial_DIN0207_L6.3mm_D2.5mm_P7.62mm_Horizontal, F.Cu at (107.2, 76.7)
- added arduino_pro_mini1: ~, custom_footprints:arduino_pro_mini_new, F.Cu at (81.0, 110.9)
- moved JP1 129.7 mm to (267.9, 26.1)
- moved JP2 129.7 mm to (266.2, 39.9)
- moved JP3 129.7 mm to (266.2, 50.4)
- moved JP6 129.7 mm to (269.1, 28.6)
- moved JP7 129.7 mm to (253.9, 56.6)
- moved JP8 129.7 mm to (265.1, 55.3)

Commit message: 4.20
Parts:
- removed JP1: FTDI Basic, 1X06
- removed JP2, JP3: , 1X02
- removed JP6, JP7: , 1X12
- removed JP8: FIDUCIALUFIDUCIAL, MICRO-FIDUCIAL
- added BME1: ~, custom_footprints:AHT20+BMP280, F.Cu at (138.0, 75.7)
- added BT3: Battery_Cell, Battery:BatteryHolder_Keystone_2460_1xAA, F.Cu at (164.4, 53.3)
- added BZ3: Buzzer, Buzzer_Beeper:Buzzer_12x9.5RM7.6, F.Cu at (133.5, 90.0)
- added R3: 100, Resistor_THT:R_Axial_DIN0207_L6.3mm_D2.5mm_P7.62mm_Horizontal, F.Cu at (145.6, 85.2)
- added R4: 100k, Resistor_THT:R_Axial_DIN0207_L6.3mm_D2.5mm_P7.62mm_Horizontal, F.Cu at (145.6, 89.3)
- added SW2: SW_Push, Button_Switch_THT:SW_PUSH_6mm, F.Cu at (148.6, 69.1)
- added TH2: Thermistor, Resistor_THT:R_Axial_DIN0207_L6.3mm_D2.5mm_P7.62mm_Horizontal, F.Cu at (145.6, 93.3)
- added U1: ~, custom_footprints:ND0205MA Voltage Regulator, F.Cu at (170.0, 103.6)
- added U2: ~, custom_footprints:Ultrasonic Sensor HC-SR04, F.Cu at (112.1, 51.0)
- added arduino_pro_mini1: ~, custom_footprints:arduino_pro_mini_new, F.Cu at (113.5, 99.6)
- moved BME280 75.9 mm to (58.7, 44.0)
- moved BZ1 75.9 mm to (7.36, 50.5)
- moved R1 75.9 mm to (10.5, 37.8)
- moved R2 75.9 mm to (47.3, 55.9)
- moved TH1 75.9 mm to (53.1, 23.5)
- moved arduino_pro_mini1 75.9 mm to (26.9, 57.7)
- moved BT2 75.9 mm to (38.6, 16.9)
- moved SW1 75.9 mm to (4.57, 25.0)
Routing:
- removed copper zone on B.Cu, net GND
- removed copper zone on F.Cu, net GND
Other:
- board text removed: "10"
- board text removed: "10MHz"
- board text removed: "11"
- board text removed: "12"
- board text removed: "13"
- board text removed: "16MHz"
- board text removed: "2"
- board text removed: "20MHz"
- board text removed: "3"
- board text removed: "3.3V"
- board text removed: "4"
- board text removed: "5"
- board text removed: "5V"
- board text removed: "6"
- board text removed: "7"
- board text removed: "8"
- board text removed: "8MHz"
- board text removed: "9"
- board text removed: "A0"
- board text removed: "A1"
- board text removed: "A2"
- board text removed: "A3"
- board text removed: "A4"
- board text removed: "A5"
- board text removed: "A6"
- board text removed: "A7"
- board text removed: "Arduino Pro"
- board text removed: "Arduino Pro Mini"
- board text removed: "BLK"
- board text removed: "GND"
- board text removed: "GRN"
- board text removed: "Mini"
- board text removed: "RAW"
- board text removed: "RST"
- board text removed: "RXI"
- board text removed: "Reset"
- board text removed: "TXO"
- board text removed: "VCC"
- board text removed: "v14"
