File: ThermoBuzzer_pcb/ThermoBuzzer_pcb.kicad_pcb (KiCad board)
At the start: 2 copper layers, 61.4 x 58.1 mm, 10 parts, among them SW2 SW_Push

Commit message: 4.22
Parts:
- moved arduino_pro_mini1 0.44 mm to (127.0, 106.0)
Connections:
- U1 pad 2: unconnected-(U1-GND-Pad2) -> GND
- U1 pad 3: unconnected-(U1-GND-Pad3) -> GND
Changed lines of the file:
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@@
 	(net 35 "unconnected-(arduino_pro_mini1-A5-Padm2)")
 	(net 36 "unconnected-(arduino_pro_mini1-6-Padl4)")
-	(net 37 "unconnected-(U1-GND-Pad3)")
-	(net 38 "unconnected-(U1-GND-Pad2)")
 	(footprint "custom_footprints:AHT20+BMP280"
 		(layer "F.Cu")
@@
 		(pad "1" thru_hole rect
 			(at -4.5 -4.08)
-			(size 1.54 1.54)
-			(drill 0.8)
+			(size 2 2)
+			(drill 1.016)
 			(layers "*.Cu" "*.Mask")
 			(remove_unused_layers no)
@@
 		(pad "2" thru_hole circle
 			(at -4.5 -1.54)
-			(size 1.524 1.524)
-			(drill 0.8)
+			(size 2 2)
+			(drill 1.016)
 			(layers "*.Cu" "*.Mask")
 			(remove_unused_layers no)
@@
 		(pad "3" thru_hole circle
 			(at -4.5 1)
-			(size 1.524 1.524)
-			(drill 0.8)
+			(size 2 2)
+			(drill 1.016)
 			(layers "*.Cu" "*.Mask")
 			(remove_unused_layers no)
@@
 		(pad "4" thru_hole circle
 			(at -4.5 3.54)
-			(size 1.524 1.524)
-			(drill 0.8)
+			(size 2 2)
+			(drill 1.016)
 			(layers "*.Cu" "*.Mask")
 			(remove_unused_layers no)
@@
 	(footprint "Resistor_THT:R_Axial_DIN0207_L6.3mm_D2.5mm_P7.62mm_Horizontal"
 		(layer "F.Cu")
-		(at 99.2 82.8)
+		(at 99.2 82.804)
 		(descr "Resistor, Axial_DIN0207 series, Axial, Horizontal, pin pitch=7.62mm, 0.25W = 1/4W, length*diameter=6.3*2.5mm^2, http://cdn-reichelt.de/documents/datenblatt/B400/1_4W%23YAG.pdf")
 		(tags "Resistor Axial_DIN0207 series Axial Horizontal pin pitch 7.62mm 0.25W = 1/4W length 6.3mm diameter 2.5mm")
@@
 		(pad "1" thru_hole rect
 			(at -17.78 7.62 90)
-			(size 2.54 2.54)
-			(drill 0.8)
+			(size 2 2)
+			(drill 1.016)
 			(layers "*.Cu" "*.Mask")
 			(remove_unused_layers no)
@@
 		(pad "2" thru_hole circle
 			(at -15.24 7.62 90)
-			(size 2.54 2.54)
-			(drill 0.8)
-			(layers "*.Cu" "*.Mask")
-			(remove_unused_layers no)
-			(net 38 "unconnected-(U1-GND-Pad2)")
+			(size 2 2)
+			(drill 1.016)
+			(layers "*.Cu" "*.Mask")
+			(remove_unused_layers no)
+			(net 1 "GND")
 			(pinfunction "GND")
 			(pintype "power_in")
@@
 		(pad "3" thru_hole circle
 			(at -12.7 7.62 90)
-			(size 2.54 2.54)
-			(drill 0.8)
-			(layers "*.Cu" "*.Mask")
-			(remove_unused_layers no)
-			(net 37 "unconnected-(U1-GND-Pad3)")
+			(size 2 2)
+			(drill 1.016)
+			(layers "*.Cu" "*.Mask")
+			(remove_unused_layers no)
+			(net 1 "GND")
 			(pinfunction "GND")
 			(pintype "power_in")
@@
 		(pad "4" thru_hole circle
 			(at -10.16 7.62 90)
-			(size 2.54 2.54)
-			(drill 0.8)
+			(size 2 2)
+			(drill 1.016)
 			(layers "*.Cu" "*.Mask")
 			(remove_unused_layers no)
@@
 		(attr smd)
 		(fp_rect
+			(start 27.5 1.6)
+			(end 43.5 13.6)
+			(stroke
+				(width 0.1)
+				(type solid)
+			)
+			(fill no)
+			(layer "F.SilkS")
+		)
+		(fp_rect
 			(start 17.78 -2.54)
 			(end 27.94 0)
@@
 		)
 		(fp_rect
+			(start 1.5 1.6)
+			(end 17.5 13.6)
+			(stroke
+				(width 0.1)
+				(type solid)
+			)
+			(fill no)
+			(layer "F.SilkS")
+		)
+		(fp_rect
 			(start 0 0)
-			(end 45 13.5)
-			(stroke
-				(width 0.1)
-				(type solid)
+			(end 45 1.6)
+			(stroke
+				(width 0.1)
+				(type default)
 			)
 			(fill no)
 			(layer "F.SilkS")
+		)
+		(fp_text user "TRIG"
+			(at 20 -7.1 180)
+			(unlocked yes)
+			(layer "F.SilkS")
+			(effects
+				(font
+					(size 1 1)
+					(thickness 0.1)
+				)
+				(justify left bottom)
+			)
+		)
+		(fp_text user "ECHO"
+			(at 22.3 -5.2 180)
+			(unlocked yes)
+			(layer "F.SilkS")
+			(effects
+				(font
+					(size 1 1)
+					(thickness 0.1)
+				)
+				(justify left bottom)
+			)
+		)
+		(fp_text user "VCC"
+			(at 17.6 -5.2 180)
+			(unlocked yes)
+			(layer "F.SilkS")
+			(effects
+				(font
+					(size 1 1)
+					(thickness 0.1)
+				)
+				(justify left bottom)
+			)
+		)
+		(fp_text user "GND"
+			(at 25.3 -6.7 180)
+			(unlocked yes)
+			(layer "F.SilkS")
+			(effects
+				(font
+					(size 1 1)
+					(thickness 0.1)
+				)
+				(justify left bottom)
+			)
 		)
 		(fp_text user "${REFERENCE}"
@@
 			(pintype "power_out")
 		)
+		(group ""
+			(members "04b22043-cf9f-4777-bf54-db2a98536750" "09eb6ae9-2dc4-46b9-b47c-c6830e340d25"
+				"1d380a97-c386-4734-aff4-5a555fa1e966" "2212bed8-4daa-4029-86e0-04c5b0238732"
+				"44420470-fd1a-48fe-b488-5aa03570ab6c" "88d44051-1b52-4097-bc89-f0306afedfe4"
+				"9f852411-fadf-4bc8-b776-af9461ab94b0" "ab7ec5d6-f614-4036-8908-9842f64b375f"
+				"bbb122a6-9a11-4a21-9a06-0282152d61d7" "c32b5dc9-36f2-4327-8ef4-8dc035506f6f"
+			)
+		)
 		(embedded_fonts no)
 	)
@@
 	(footprint "custom_footprints:arduino_pro_mini_new"
 		(layer "F.Cu")
-		(at 127.2416 105.6803 90)
+		(at 127 106.045 90)
 		(property "Reference" "arduino_pro_mini1"
 			(at -4.8768 1.9558 90)
