File: ThermoBuzzer_pcb/ThermoBuzzer_pcb.kicad_pcb (KiCad board)
At the start: 2 copper layers, 60 x 60 mm, 13 parts, among them SW2 SW_Push

Commit message: 5.1
Parts:
- R3: value 100 -> 4.7k
- moved U3 19.5 mm to (134.5, 88.3)
