File: ThermoBuzzer_pcb/ThermoBuzzer_pcb_final.kicad_pcb (KiCad board)
At the start: 2 copper layers, 60 x 60 mm, 13 parts, among them SW2 SW_Push

Commit message: 4.27
Parts:
- removed ? (x3): , 
- BT3: footprint custom_footprints:6s-aa 14500 -> Battery:BatteryHolder_Keystone_2460_1xAA
- moved BT3 9.10 mm to (98.5, 118.3)
Routing:
- net +1.5V: track 50.0 -> 48.5 mm
- net (no net): vias 1 -> 0
Other:
- board size 60 x 60 mm -> 61 x 59.7 mm
