File: ThermoBuzzer_pcb/_autosave-ThermoBuzzer_pcb.kicad_sch (KiCad schematic)
At the start: 10 parts, among them SW2 SW_Push

Commit message: 4.27
Parts:
- BT3: footprint Battery:BatteryHolder_Keystone_2460_1xAA -> custom_footprints:6s-aa 14500
Changed lines of the file:
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@@
 			)
 		)
-		(property "Footprint" "Battery:BatteryHolder_Keystone_2460_1xAA"
+		(property "Footprint" "custom_footprints:6s-aa 14500"
 			(at 107.95 100.076 90)
 			(effects
