File: ThermoBuzzer_pcb/backups/ThermoBuzzer_pcb_finalfinal.kicad_pcb (KiCad board)
At the start: 2 copper layers, 60 x 60 mm, 13 parts, among them SW2 SW_Push

Commit message: 5.11
Parts:
- moved ? 1.45 mm to (118.0, 74.1)
- moved U2 1.28 mm to (140.5, 83.5)
- moved ? 0.48 mm to (99.8, 86.3)
Routing:
- net +3.3V: track 152.5 -> 141.0 mm
- net Net-(U1-A2): track 25.9 -> 24.2 mm
- net GND: track 104.8 -> 103.2 mm
- net Net-(U1-11): track 10.5 -> 9.26 mm
- net Net-(U1-10): track 15.2 -> 13.9 mm
- net Net-(U1-A1): track 23.6 -> 22.3 mm
- net Net-(U4-GND): track 36.1 -> 37.3 mm
